File: Capteurs_PCB/Capteurs_PCB.kicad_sch (KiCad schematic)
At the start: 11 parts, among them J1 Batterie, J2 RaspberryPi, J3 Prop1, J4 Prop2, J5 Alim_Prop1, J6 Alim_Prop2, J7 Moteur_seringues_1, J8 Moteur_seringues_2, J9 LED, U7 ZXBM5210-SP, U8 ZXBM5210-SP

Commit message: update pcb
Parts:
- removed J1: Batterie, Connector_Hirose:Hirose_DF13-02P-1.25DSA_1x02_P1.25mm_Vertical, symbol Connector:Conn_01x02_Socket
- removed J2: RaspberryPi, Connector_PinSocket_2.54mm:PinSocket_1x02_P2.54mm_Vertical, symbol Connector:Conn_01x02_Socket
- removed J7: Moteur_seringues_1, Connector_PinSocket_2.54mm:PinSocket_1x02_P2.54mm_Vertical, symbol Connector:Conn_01x02_Socket
- removed J8: Moteur_seringues_2, Connector_PinSocket_2.54mm:PinSocket_1x02_P2.54mm_Vertical, symbol Connector:Conn_01x02_Socket
- removed U7, U8: ZXBM5210-SP, Package_SO:Diodes_SO-8EP, symbol Driver_Motor:ZXBM5210-SP
- added C101, C102, C103, C104, C105, C106: 100n, symbol Device:C_Small
- added C107: 4u7, symbol Device:C_Small
- added H101, H102, H103, H104: MountingHole_Pad, symbol Mechanical:MountingHole_Pad
- added J101: Conn_01x03, symbol Connector_Generic:Conn_01x03
- added J102: Conn_01x02, symbol Connector_Generic:Conn_01x02
- added J103: Conn_02x20_Odd_Even, symbol Connector_Generic:Conn_02x20_Odd_Even
- added J104: Conn_ST_STDC14, symbol Connector:Conn_ST_STDC14
- added SW101: SW_DPDT_x2, symbol Switch:SW_DPDT_x2
- added U101: STM32L476RGTx, Package_QFP:LQFP-64_10x10mm_P0.5mm, symbol MCU_ST_STM32L4:STM32L476RGTx
Connections:
- net Earth: now also H101.1, H102.1, H103.1, H104.1, J101.1 (Pin_1), J102.1 (Pin_1), J103.14 (Pin_14), J103.20 (Pin_20), J103.25 (Pin_25), J103.30 (Pin_30), J103.34 (Pin_34), J103.39 (Pin_39), J103.6 (Pin_6), J103.9 (Pin_9), U101.12 (VSSA), U101.18 (VSS), U101.31 (VSS), U101.47 (VSS), U101.63 (VSS)
- net FWD1: now also U101.16 (PA2)
- net FWD2: now also U101.41 (PA8)
- net REV1: now also U101.17 (PA3)
- net REV2: now also U101.42 (PA9)
- net SigProp1: now also U101.56 (PB4)
- net SigProp2: now also U101.58 (PB6)
- net Sig_LED: now also U101.43 (PA10)
- net UART_RX: now also U101.52 (PC11)
- net UART_TX: now also U101.51 (PC10)
- net VDD_LED: no longer J3.2 (Pin_2), J4.2 (Pin_2)
- net V_12V renamed V_ALIM_PROP
- new net: J104.5 (GND), J104.7 (GND)
- new net +5V: C101.1, C102.1, C103.1, C104.1, C105.1, C106.1, C107.1, J103.2 (Pin_2), J103.4 (Pin_4), U101.1 (VBAT), U101.13 (VDDA), U101.19 (VDD), U101.32 (VDD), U101.48 (VDDUSB), U101.64 (VDD)
- new net +BATT: J102.2 (Pin_2), SW101.2 (B)
- new net CS: U101.35 (PB14)
- new net GND: C101.2, C102.2, C103.2, C104.2, C105.2, C106.2, C107.2
- new net INT1: U101.14 (PA0)
- new net INT2: U101.15 (PA1)
- new net MISO: U101.22 (PA6)
- new net MOSI: U101.23 (PA7)
- new net RPI_UART_RX: J103.10 (Pin_10)
- new net RPI_UART_TX: J103.8 (Pin_8)
- new net Regulation/Vin: SW101.1 (A)
- new net SCLK: U101.21 (PA5)
- new net SDX: U101.36 (PB15)
- new net SS: U101.20 (PA4)
- no-connect marks 0 -> 64
Other:
- removed sheet Microcontrolleur
- sheet Regulation ports: added 3.3V, 5.1V, 7.4V, Vin; removed none
- note removed: "Batterie"
- note removed: "Moteurs seringues"
- moved on the sheet: J9
