File: Capteurs_PCB/Capteurs_PCB.kicad_pcb (KiCad board)
At the start: 2 copper layers, 56 parts, among them J1 Conn_01x04, J101 Conn_01x03, J103 Conn_02x20_Odd_Even, J104 Conn_ST_STDC14, J2 Conn_01x03, J3 Alim_Prop1, J4 Conn_01x02, J5 Alim_Prop1, J6 Conn_01x03, J7 Conn_01x03, SW101 SW_DPDT_x2, U1 STM32L412KBTx, U3 LSM6DSL, U6 32350268

Commit message: Start routage
Parts:
- moved J1 85.2 mm to (180.4, 124.4)
- moved J101 85.2 mm to (189.7, 114.7)
- moved J104 85.2 mm to (196.2, 123.8)
- moved J3 85.2 mm to (193.8, 87.0)
- moved J5 85.2 mm to (193.8, 92.5)
- moved J6 85.2 mm to (180.4, 114.7)
- moved J7 85.2 mm to (185.1, 114.7)
- moved J4 85.2 mm to (198.2, 102.5)
- moved C1 78.0 mm to (112.5, 191.9)
- moved C101 78.0 mm to (93.9, 151.5)
- moved C102 78.0 mm to (93.9, 154.8)
- moved C103 78.0 mm to (93.9, 158.2)
- moved C107 78.0 mm to (93.9, 161.6)
- moved C2 78.0 mm to (93.9, 141.4)
- moved C3 78.0 mm to (93.9, 144.8)
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Routing:
- added copper zone on B.Cu, net (none)
- added copper zone on F.Cu, net (none)
Other:
- board outline added: 89 x 72 mm

Commit message: Update routage
Parts:
- J3: value Alim_Prop1 -> Alim_Prop2
- moved J7 102.1 mm to (98.9, 60.0), turned to 90 degrees
- moved R409 98.3 mm to (141.5, 68.9), turned to 90 degrees
- moved U6 97.4 mm to (125.0, 88.9)
- moved R408 95.8 mm to (139.0, 68.9), turned to 90 degrees
- moved U3 95.4 mm to (134.8, 87.8), turned to -90 degrees
- moved R407 93.3 mm to (136.5, 68.9), turned to 90 degrees
- moved J5 90.7 mm to (108.8, 124.0)
- moved J1 86.1 mm to (94.4, 124.0), turned to 90 degrees
- moved U402 84.6 mm to (149.0, 69.0), turned to 90 degrees
- moved J6 84.6 mm to (115.9, 60.0), turned to 90 degrees
- moved D401 83.1 mm to (132.5, 61.0)
- moved D402 83.1 mm to (140.0, 61.0)
- moved D403 83.1 mm to (147.5, 61.0)
- moved U401 78.9 mm to (149.0, 76.1), turned to 90 degrees
- moved U2 74.1 mm to (149.0, 83.2), turned to 90 degrees
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
Commit message: Routage en cours
Parts:
- C1, C101, C102, C103, C107, C2, C3, C4, C401, C405, C6, C7, C9: footprint Capacitor_SMD:C_1206_3216Metric_Pad1.33x1.80mm_HandSolder -> Capacitor_SMD:C_0603_1608Metric_Pad1.08x0.95mm_HandSolder
- moved SW101 83.3 mm to (139.6, 79.0), turned to -90 degrees
- moved C107 82.6 mm to (144.1, 96.0)
- moved C103 82.2 mm to (144.0, 93.0)
- moved C102 81.1 mm to (144.0, 91.0)
- moved C101 80.1 mm to (144.0, 89.0)
- moved L1 68.7 mm to (134.0, 103.0), turned to 90 degrees
- moved C4 63.8 mm to (139.0, 103.0), turned to -90 degrees
- moved C3 60.0 mm to (137.0, 103.0), turned to -90 degrees
- moved C2 51.0 mm to (134.0, 110.0), turned to 180 degrees
- moved U2 1.80 mm to (149.0, 85.0)
- moved U401 0.17 mm to (149.0, 76.3)

Commit message: Suite
Parts:
- moved C7 116.8 mm to (98.1, 71.8), turned to 90 degrees
- moved C1 115.0 mm to (97.3, 78.0), turned to -90 degrees
- moved C6 114.9 mm to (91.4, 72.1), turned to 90 degrees
- moved C405 107.9 mm to (134.1, 68.9), turned to 180 degrees
- moved C404 96.8 mm to (140.0, 80.0)
- moved C5 93.4 mm to (141.0, 69.9)
- moved C401 92.5 mm to (134.1, 81.0), turned to 180 degrees
- moved R2 92.4 mm to (127.0, 69.9), turned to 90 degrees
- moved R1 89.8 mm to (129.0, 69.9), turned to -90 degrees
- moved R403 87.5 mm to (130.0, 79.9), turned to -90 degrees
- moved R404 85.9 mm to (137.0, 73.8), turned to 90 degrees
- moved R402 85.1 mm to (128.0, 79.9), turned to 90 degrees
- moved C406 83.5 mm to (121.0, 76.9), turned to 180 degrees
- moved C403 77.5 mm to (141.0, 93.0)
- moved R401 77.3 mm to (137.0, 84.9), turned to 90 degrees
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
Commit message: Début de routage
Parts:
- D401, D402, D403: footprint LED_THT:LED_D5.0mm_Clear -> LED_SMD:LED_0402_1005Metric_Pad0.77x0.64mm_HandSolder
- moved J103 48.0 mm to (76.7, 115.9), turned to 180 degrees
- moved U6 9.27 mm to (102.5, 86.1), turned to -90 degrees
- moved J104 7.12 mm to (113.4, 123.3), turned to 90 degrees
- moved D401 1.54 mm to (134.0, 61.0), turned to 180 degrees
- moved D403 1.46 mm to (146.0, 61.0), turned to -90 degrees
- moved C1 0.86 mm to (98.2, 78.0)
- moved C6 0.86 mm to (92.2, 72.1)
- turned D402 to 180 degrees
- turned C2 to 0 degrees
- turned C7 to -90 degrees
Connections:
- J3 pad 2: /V_ALIM_PROP -> (no net)
- J5 pad 2: /V_ALIM_PROP -> (no net)
Routing:
- net +3.3V: track 0.00 -> 93.2 mm
- net ST_TX: track 0.00 -> 36.2 mm, vias 0 -> 2
- net SWDIO: track 0.00 -> 35.4 mm, vias 0 -> 2
- net SWCLK: track 0.00 -> 33.0 mm, vias 0 -> 2
- net NRST: track 0.00 -> 32.5 mm, vias 0 -> 2
- net SWO: track 0.00 -> 31.8 mm, vias 0 -> 2
- net /Sig_LED: track 0.00 -> 26.9 mm, vias 0 -> 2
- net +3V3: track 0.00 -> 19.8 mm
- net MISO: track 0.00 -> 16.9 mm
- net /RPI_UART_RX: track 0.00 -> 16.5 mm, vias 0 -> 2
- net /RPI_UART_TX: track 0.00 -> 16.4 mm
- net SS: track 0.00 -> 10.7 mm
- net MOSI: track 0.00 -> 10.6 mm
- net SCLK: track 0.00 -> 10.1 mm, vias 0 -> 2
- net +3.3VA: track 0.00 -> 9.53 mm
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- added copper zone on B.Cu, net GND
- added copper zone on F.Cu, net GND
- removed copper zone on F.Cu, net (none)

Commit message: Problème réglé
Parts:
- removed the C1 at (98.2, 78.0)
- removed the C101 at (104.8, 105.7)
- removed the C102 at (106.8, 105.7)
- removed the C103 at (108.8, 105.7)
- removed the C107 at (111.8, 105.5)
- removed the C2 at (105.0, 102.8)
- removed the C3 at (107.6, 99.7)
- removed the C4 at (109.6, 99.7)
- removed the C401 at (134.1, 81.0)
- removed the C402 at (121.0, 88.0)
- removed the C403 at (141.0, 93.0)
- removed the C404 at (140.0, 80.0)
- removed the C405 at (134.1, 68.9)
- removed the C406 at (121.0, 76.9)
- removed the C5 at (141.0, 69.9)
- removed the C6 at (92.2, 72.1)
- removed the C7 at (98.1, 71.8)
- removed the C8 at (121.0, 99.9)
- removed the C9 at (135.0, 92.9)
- removed the D401 at (134.0, 61.0)
- removed the D402 at (140.0, 61.0)
- removed the D403 at (146.0, 61.0)
- removed the H101 at (78.0, 61.0)
- removed the H102 at (78.0, 123.0)
- removed the H103 at (157.0, 61.0)
- removed the H104 at (157.0, 123.0)
- removed the J1 at (87.4, 123.0)
- removed the J101 at (159.0, 104.5)
- removed the J103 at (76.7, 115.9)
- removed the J104 at (113.4, 123.3)
- removed the J2 at (134.9, 124.0)
- removed the J3 at (146.8, 124.0)
- removed the J4 at (159.0, 81.5)
- removed the J5 at (101.8, 123.0)
- removed the J6 at (115.9, 60.0)
- removed the J7 at (98.9, 60.0)
- removed the L1 at (104.6, 99.7)
- removed the R1 at (129.0, 69.9)
- removed the R2 at (127.0, 69.9)
- removed the R3 at (129.0, 91.9)
- removed the R4 at (137.0, 96.9)
- removed the R401 at (137.0, 84.9)
- removed the R402 at (128.0, 79.9)
- removed the R403 at (130.0, 79.9)
- removed the R404 at (137.0, 73.8)
- removed the R407 at (125.0, 71.9)
- removed the R408 at (125.0, 83.0)
- removed the R409 at (125.0, 94.9)
- removed the R5 at (131.0, 91.9)
- removed the SW101 at (150.8, 79.0)
- removed the U1 at (96.8, 100.8)
- removed the U3 at (95.3, 72.1)
- added C1: 100nF, Capacitor_SMD:C_0603_1608Metric_Pad1.08x0.95mm_HandSolder, F.Cu at (54.0, 59.3)
- added C1: 100nF, Capacitor_SMD:C_0603_1608Metric_Pad1.08x0.95mm_HandSolder, F.Cu at (107.2, 65.9)
- added C101: 100n, Capacitor_SMD:C_0603_1608Metric_Pad1.08x0.95mm_HandSolder, F.Cu at (38.0, 29.4)
- added C101: 100n, Capacitor_SMD:C_0603_1608Metric_Pad1.08x0.95mm_HandSolder, F.Cu at (119.0, 81.0)
- added C102: 100n, Capacitor_SMD:C_0603_1608Metric_Pad1.08x0.95mm_HandSolder, F.Cu at (38.0, 31.9)
- added C102: 100n, Capacitor_SMD:C_0603_1608Metric_Pad1.08x0.95mm_HandSolder, F.Cu at (121.0, 81.0)
- added C103: 100n, Capacitor_SMD:C_0603_1608Metric_Pad1.08x0.95mm_HandSolder, F.Cu at (123.0, 81.0)
- added C103: 100n, Capacitor_SMD:C_0603_1608Metric_Pad1.08x0.95mm_HandSolder, F.Cu at (38.0, 34.4)
- added C107: 4u7, Capacitor_SMD:C_0603_1608Metric_Pad1.08x0.95mm_HandSolder, F.Cu at (38.0, 36.9)
- added C107: 4u7, Capacitor_SMD:C_0603_1608Metric_Pad1.08x0.95mm_HandSolder, F.Cu at (126.0, 80.9)
- added C2: 100n, Capacitor_SMD:C_0603_1608Metric_Pad1.08x0.95mm_HandSolder, F.Cu at (38.0, 21.8)
- added C2: 100n, Capacitor_SMD:C_0603_1608Metric_Pad1.08x0.95mm_HandSolder, F.Cu at (119.2, 78.2)
- added C3: 1u, Capacitor_SMD:C_0603_1608Metric_Pad1.08x0.95mm_HandSolder, F.Cu at (38.0, 24.3)
- added C3: 1u, Capacitor_SMD:C_0603_1608Metric_Pad1.08x0.95mm_HandSolder, F.Cu at (121.8, 75.0)
- added C4: 100n, Capacitor_SMD:C_0603_1608Metric_Pad1.08x0.95mm_HandSolder, F.Cu at (123.8, 75.0)
- added C4: 100n, Capacitor_SMD:C_0603_1608Metric_Pad1.08x0.95mm_HandSolder, F.Cu at (38.0, 26.8)
- added C401: 1u, Capacitor_SMD:C_0603_1608Metric_Pad1.08x0.95mm_HandSolder, F.Cu at (124.4, 98.6)
- added C401: 1u, Capacitor_SMD:C_0603_1608Metric_Pad1.08x0.95mm_HandSolder, F.Cu at (73.6, 24.3)
- added C402: 47u, Capacitor_SMD:CP_Elec_6.3x5.4, F.Cu at (57.1, 32.8)
- added C402: 47u, Capacitor_SMD:CP_Elec_6.3x5.4, F.Cu at (111.3, 105.6)
- added C403: 10u, Capacitor_SMD:CP_Elec_5x5.4, F.Cu at (131.3, 110.6)
- added C403: 10u, Capacitor_SMD:CP_Elec_5x5.4, F.Cu at (66.9, 30.8)
- added C404: 10u, Capacitor_SMD:CP_Elec_5x5.4, F.Cu at (130.6, 97.1)
- added C404: 10u, Capacitor_SMD:CP_Elec_5x5.4, F.Cu at (66.9, 37.7)
- added C405: 1u, Capacitor_SMD:C_0603_1608Metric_Pad1.08x0.95mm_HandSolder, F.Cu at (124.4, 86.5)
- added C405: 1u, Capacitor_SMD:C_0603_1608Metric_Pad1.08x0.95mm_HandSolder, F.Cu at (73.6, 26.8)
- added C406: 47u, Capacitor_SMD:CP_Elec_6.3x5.4, F.Cu at (111.3, 94.5)
- added C406: 47u, Capacitor_SMD:CP_Elec_6.3x5.4, F.Cu at (57.1, 40.9)
- added C5: 10u, Capacitor_SMD:CP_Elec_5x5.4, F.Cu at (131.3, 87.5)
- added C5: 10u, Capacitor_SMD:CP_Elec_5x5.4, F.Cu at (66.9, 24.0)
- added C6: 100n, Capacitor_SMD:C_0603_1608Metric_Pad1.08x0.95mm_HandSolder, F.Cu at (54.0, 52.3)
- added C6: 100n, Capacitor_SMD:C_0603_1608Metric_Pad1.08x0.95mm_HandSolder, F.Cu at (104.1, 65.9)
- added C7: 100n, Capacitor_SMD:C_0603_1608Metric_Pad1.08x0.95mm_HandSolder, F.Cu at (54.0, 54.8)
- added C7: 100n, Capacitor_SMD:C_0603_1608Metric_Pad1.08x0.95mm_HandSolder, F.Cu at (105.7, 65.9)
- added C8: 47u, Capacitor_SMD:CP_Elec_6.3x5.4, F.Cu at (110.4, 116.3)
- added C8: 47u, Capacitor_SMD:CP_Elec_6.3x5.4, F.Cu at (57.1, 24.6)
- added C9: 1u, Capacitor_SMD:C_0603_1608Metric_Pad1.08x0.95mm_HandSolder, F.Cu at (73.6, 21.8)
- added C9: 1u, Capacitor_SMD:C_0603_1608Metric_Pad1.08x0.95mm_HandSolder, F.Cu at (125.3, 110.5)
- added D401: LED, LED_SMD:LED_0402_1005Metric_Pad0.77x0.64mm_HandSolder, F.Cu at (73.3, 34.1)
- added D401: LED, LED_SMD:LED_0402_1005Metric_Pad0.77x0.64mm_HandSolder, F.Cu at (113.6, 87.9)
- added D402: LED, LED_SMD:LED_0402_1005Metric_Pad0.77x0.64mm_HandSolder, F.Cu at (113.0, 99.9)
- added D402: LED, LED_SMD:LED_0402_1005Metric_Pad0.77x0.64mm_HandSolder, F.Cu at (73.3, 36.1)
- added D403: LED, LED_SMD:LED_0402_1005Metric_Pad0.77x0.64mm_HandSolder, F.Cu at (113.5, 111.2)
- added D403: LED, LED_SMD:LED_0402_1005Metric_Pad0.77x0.64mm_HandSolder, F.Cu at (73.3, 38.1)
- added H101: MountingHole_Pad, MountingHole:MountingHole_3.2mm_M3_DIN965_Pad, F.Cu at (32.3, 24.1)
- added H101: MountingHole_Pad, MountingHole:MountingHole_3.2mm_M3_DIN965_Pad, F.Cu at (98.5, 58.5)
- added H102: MountingHole_Pad, MountingHole:MountingHole_3.2mm_M3_DIN965_Pad, F.Cu at (98.5, 120.5)
- added H102: MountingHole_Pad, MountingHole:MountingHole_3.2mm_M3_DIN965_Pad, F.Cu at (32.3, 31.3)
- added H103: MountingHole_Pad, MountingHole:MountingHole_3.2mm_M3_DIN965_Pad, F.Cu at (141.5, 58.5)
- added H103: MountingHole_Pad, MountingHole:MountingHole_3.2mm_M3_DIN965_Pad, F.Cu at (32.3, 38.4)
- added H104: MountingHole_Pad, MountingHole:MountingHole_3.2mm_M3_DIN965_Pad, F.Cu at (141.5, 120.5)
- added H104: MountingHole_Pad, MountingHole:MountingHole_3.2mm_M3_DIN965_Pad, F.Cu at (32.3, 45.6)
- added J1: Conn_01x04, Connector_PinSocket_2.54mm:PinSocket_1x04_P2.54mm_Vertical, F.Cu at (114.2, 57.8)
- added J1: Conn_01x04, Connector_PinSocket_2.54mm:PinSocket_1x04_P2.54mm_Vertical, F.Cu at (42.5, 22.9)
- added J101: Conn_01x03, Connector_PinHeader_2.54mm:PinHeader_1x03_P2.54mm_Vertical, F.Cu at (47.5, 40.5)
- added J101: Conn_01x03, Connector_PinHeader_2.54mm:PinHeader_1x03_P2.54mm_Vertical, F.Cu at (98.5, 99.1)
- added J103: Conn_02x20_Odd_Even, Connector_PinSocket_2.54mm:PinSocket_2x20_P2.54mm_Vertical, F.Cu at (26.4, 22.9)
- added J103: Conn_02x20_Odd_Even, Connector_PinSocket_2.54mm:PinSocket_2x20_P2.54mm_Vertical, F.Cu at (140.0, 114.0)
- added J104: Conn_ST_STDC14, Connector_PinHeader_1.27mm:PinHeader_2x07_P1.27mm_Vertical, F.Cu at (42.3, 50.8)
- added J104: Conn_ST_STDC14, Connector_PinHeader_1.27mm:PinHeader_2x07_P1.27mm_Vertical, F.Cu at (99.5, 79.7)
- added J2: Conn_01x03, Connector_PinSocket_2.54mm:PinSocket_1x03_P2.54mm_Vertical, F.Cu at (98.7, 89.1)
- added J2: Conn_01x03, Connector_PinSocket_2.54mm:PinSocket_1x03_P2.54mm_Vertical, F.Cu at (47.1, 22.9)
- added J3: Alim_Prop2, Connector_Hirose:Hirose_DF13-02P-1.25DSA_1x02_P1.25mm_Vertical, F.Cu at (31.2, 63.8)
- added J3: Alim_Prop2, Connector_Hirose:Hirose_DF13-02P-1.25DSA_1x02_P1.25mm_Vertical, F.Cu at (99.0, 114.2)
- added J4: Conn_01x02, Connector_PinHeader_2.54mm:PinHeader_1x02_P2.54mm_Vertical, F.Cu at (37.2, 68.5)
- added J4: Conn_01x02, Connector_PinHeader_2.54mm:PinHeader_1x02_P2.54mm_Vertical, F.Cu at (125.9, 57.7)
- added J5: Alim_Prop1, Connector_Hirose:Hirose_DF13-02P-1.25DSA_1x02_P1.25mm_Vertical, F.Cu at (99.1, 106.3)
- added J5: Alim_Prop1, Connector_Hirose:Hirose_DF13-02P-1.25DSA_1x02_P1.25mm_Vertical, F.Cu at (31.2, 69.2)
- added J6: Conn_01x03, Connector_PinHeader_2.54mm:PinHeader_1x03_P2.54mm_Vertical, F.Cu at (104.9, 57.9)
- added J6: Conn_01x03, Connector_PinHeader_2.54mm:PinHeader_1x03_P2.54mm_Vertical, F.Cu at (38.2, 40.5)
- added J7: Conn_01x03, Connector_PinHeader_2.54mm:PinHeader_1x03_P2.54mm_Vertical, F.Cu at (42.8, 40.5)
- added J7: Conn_01x03, Connector_PinHeader_2.54mm:PinHeader_1x03_P2.54mm_Vertical, F.Cu at (98.7, 68.9)
- added L1: 39n, Inductor_SMD:L_0805_2012Metric_Pad1.05x1.20mm_HandSolder, F.Cu at (118.8, 75.0)
- added L1: 39n, Inductor_SMD:L_0805_2012Metric_Pad1.05x1.20mm_HandSolder, F.Cu at (42.0, 67.5)
- added R1: 402k, Resistor_SMD:R_0603_1608Metric_Pad0.98x0.95mm_HandSolder, F.Cu at (119.3, 87.5)
- added R1: 30.1k, Resistor_SMD:R_0603_1608Metric_Pad0.98x0.95mm_HandSolder, F.Cu at (73.6, 29.4)
- added R2: 52.2k, Resistor_SMD:R_0603_1608Metric_Pad0.98x0.95mm_HandSolder, F.Cu at (117.3, 87.5)
- added R2: 402k, Resistor_SMD:R_0603_1608Metric_Pad0.98x0.95mm_HandSolder, F.Cu at (73.6, 31.9)
- added R3: 402k, Resistor_SMD:R_0603_1608Metric_Pad0.98x0.95mm_HandSolder, F.Cu at (77.9, 21.8)
- added R3: 140, Resistor_SMD:R_0603_1608Metric_Pad0.98x0.95mm_HandSolder, F.Cu at (119.3, 109.5)
- added R4: 5.6k, Resistor_SMD:R_0603_1608Metric_Pad0.98x0.95mm_HandSolder, F.Cu at (127.3, 114.5)
- added R4: 5.6k, Resistor_SMD:R_0603_1608Metric_Pad0.98x0.95mm_HandSolder, F.Cu at (77.9, 24.3)
- added R401: 5.6k, Resistor_SMD:R_0603_1608Metric_Pad0.98x0.95mm_HandSolder, F.Cu at (127.3, 102.5)
- added R401: 5.6k, Resistor_SMD:R_0603_1608Metric_Pad0.98x0.95mm_HandSolder, F.Cu at (77.9, 29.4)
- added R402: 402k, Resistor_SMD:R_0603_1608Metric_Pad0.98x0.95mm_HandSolder, F.Cu at (77.9, 31.9)
- added R402: 80.4, Resistor_SMD:R_0603_1608Metric_Pad0.98x0.95mm_HandSolder, F.Cu at (118.3, 97.5)
- added R403: 80.4k, Resistor_SMD:R_0603_1608Metric_Pad0.98x0.95mm_HandSolder, F.Cu at (82.3, 21.8)
- added R403: 402k, Resistor_SMD:R_0603_1608Metric_Pad0.98x0.95mm_HandSolder, F.Cu at (120.3, 97.5)
- added R404: 5.6k, Resistor_SMD:R_0603_1608Metric_Pad0.98x0.95mm_HandSolder, F.Cu at (82.3, 24.3)
- added R404: 5.6k, Resistor_SMD:R_0603_1608Metric_Pad0.98x0.95mm_HandSolder, F.Cu at (127.3, 91.4)
- added R407: 300, Resistor_SMD:R_0603_1608Metric_Pad0.98x0.95mm_HandSolder, F.Cu at (82.3, 26.8)
- added R407: 300, Resistor_SMD:R_0603_1608Metric_Pad0.98x0.95mm_HandSolder, F.Cu at (115.3, 89.5)
- added R408: 300, Resistor_SMD:R_0603_1608Metric_Pad0.98x0.95mm_HandSolder, F.Cu at (82.3, 29.4)
- added R408: 300, Resistor_SMD:R_0603_1608Metric_Pad0.98x0.95mm_HandSolder, F.Cu at (114.8, 100.5)
- added R409: 300, Resistor_SMD:R_0603_1608Metric_Pad0.98x0.95mm_HandSolder, F.Cu at (115.3, 112.5)
- added R409: 300, Resistor_SMD:R_0603_1608Metric_Pad0.98x0.95mm_HandSolder, F.Cu at (82.3, 31.9)
- added R5: 402k, Resistor_SMD:R_0603_1608Metric_Pad0.98x0.95mm_HandSolder, F.Cu at (121.3, 109.5)
- added R5: 140k, Resistor_SMD:R_0603_1608Metric_Pad0.98x0.95mm_HandSolder, F.Cu at (77.9, 26.8)
- added SW101: SW_DPDT_x2, Button_Switch_SMD:SW_DPDT_CK_JS202011JCQN, F.Cu at (133.5, 78.0)
- added SW101: SW_DPDT_x2, Button_Switch_SMD:SW_DPDT_CK_JS202011JCQN, F.Cu at (40.2, 63.4)
- added U1: STM32L412KBTx, Package_QFP:LQFP-32_7x7mm_P0.8mm, F.Cu at (34.4, 54.9)
- added U1: STM32L412KBTx, Package_QFP:LQFP-32_7x7mm_P0.8mm, F.Cu at (112.1, 77.8)
- added U3: LSM6DSL, Package_LGA:LGA-14_3x2.5mm_P0.5mm_LayoutBorder3x4y, F.Cu at (54.1, 49.0)
- added U3: LSM6DSL, Package_LGA:LGA-14_3x2.5mm_P0.5mm_LayoutBorder3x4y, F.Cu at (110.6, 65.8)
- moved U6 25.8 mm to (117.5, 65.1), turned to 0 degrees
- moved U2 20.1 mm to (121.3, 115.5)
- moved U401 20.1 mm to (121.3, 103.5)
- moved U402 20.1 mm to (121.3, 92.5)
Connections:
- U402 pad 6: +7.5V -> (no net)
Routing:
- net +3.3V: track 93.2 -> 0.21 mm
- net ST_TX: track 36.2 -> 0.00 mm, vias 2 -> 0
- net SWDIO: track 35.4 -> 0.00 mm, vias 2 -> 0
- net SWCLK: track 33.0 -> 0.00 mm, vias 2 -> 0
- net NRST: track 32.5 -> 0.00 mm, vias 2 -> 0
- net SWO: track 31.8 -> 0.00 mm, vias 2 -> 0
- net /Sig_LED: track 26.9 -> 0.00 mm, vias 2 -> 0
- net +3V3: track 19.8 -> 0.00 mm
- net MISO: track 16.9 -> 0.00 mm
- net /RPI_UART_RX: track 16.5 -> 0.00 mm, vias 2 -> 0
- net /RPI_UART_TX: track 16.4 -> 0.00 mm
- net SS: track 10.7 -> 0.00 mm
- net MOSI: track 10.6 -> 0.00 mm
- net SCLK: track 10.1 -> 0.00 mm, vias 2 -> 0
- net +3.3VA: track 9.53 -> 0.41 mm
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- removed copper zone on B.Cu, net (none)
- removed copper zone on B.Cu, net GND
- removed copper zone on F.Cu, net GND
Other:
- board size 89 x 72 mm -> 51 x 70 mm

Commit message: modif kicad
Parts:
- removed the H101 at (98.5, 58.5)
- removed the H102 at (98.5, 120.5)
- removed the H103 at (141.5, 58.5)
- removed the H104 at (141.5, 120.5)
- removed the J1 at (114.2, 57.8)
- removed the J101 at (98.5, 99.1)
- removed the J103 at (140.0, 114.0)
- removed the J104 at (99.5, 79.7)
- removed the J2 at (98.7, 89.1)
- removed the J3 at (99.0, 114.2)
- removed the J4 at (125.9, 57.7)
- removed the J5 at (99.1, 106.3)
- removed the J6 at (104.9, 57.9)
- removed the J7 at (98.7, 68.9)
- removed the U1 at (112.1, 77.8)
- moved J103 146.8 mm to (146.0, 108.0), turned to 180 degrees
- moved H104 135.2 mm to (148.0, 115.5)
- moved H103 116.7 mm to (148.0, 53.5)
- moved H102 111.3 mm to (105.0, 115.5)
- moved J4 96.7 mm to (132.7, 53.0), turned to 90 degrees
- moved J3 86.8 mm to (105.5, 108.8), turned to 90 degrees
- moved U1 85.9 mm to (118.5, 72.5), turned to 180 degrees
- moved J2 84.6 mm to (105.0, 84.6), turned to 180 degrees
- moved J1 83.7 mm to (120.7, 53.0), turned to 90 degrees
- moved J5 81.1 mm to (105.5, 101.8), turned to 90 degrees
- moved J101 78.9 mm to (105.0, 94.5), turned to 180 degrees
- moved H101 78.4 mm to (105.0, 53.4)
- moved J6 74.3 mm to (111.4, 53.0), turned to 90 degrees
- moved J104 68.2 mm to (106.0, 75.1), turned to 180 degrees
- moved J7 66.3 mm to (105.0, 63.5), turned to 180 degrees
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
Commit message: Suite PCB
Parts:
- removed the C1 at (113.7, 60.9)
- removed the C101 at (125.5, 76.0)
- removed the C102 at (127.5, 76.0)
- removed the C103 at (129.5, 76.0)
- removed the C107 at (132.5, 75.9)
- removed the C2 at (125.6, 73.2)
- removed the C3 at (128.3, 70.0)
- removed the C4 at (130.3, 70.0)
- removed the C401 at (130.9, 93.6)
- removed the C402 at (117.8, 100.6)
- removed the C403 at (137.8, 105.6)
- removed the C404 at (137.1, 92.1)
- removed the C405 at (130.9, 81.5)
- removed the C406 at (117.8, 89.5)
- removed the C5 at (137.8, 82.5)
- removed the C6 at (110.6, 60.9)
- removed the C7 at (112.1, 60.9)
- removed the C8 at (116.9, 111.4)
- removed the C9 at (131.8, 105.5)
- removed the D401 at (120.1, 82.9)
- removed the D402 at (119.4, 95.0)
- removed the D403 at (120.0, 106.2)
- removed the L1 at (125.3, 70.0)
- removed the R1 at (125.8, 82.5)
- removed the R2 at (123.8, 82.5)
- removed the R3 at (125.8, 104.5)
- removed the R4 at (133.8, 109.5)
- removed the R401 at (133.8, 97.5)
- removed the R402 at (124.8, 92.5)
- removed the R403 at (126.8, 92.5)
- removed the R404 at (133.8, 86.4)
- removed the R407 at (121.8, 84.5)
- removed the R408 at (121.3, 95.5)
- removed the R409 at (121.8, 107.5)
- removed the R5 at (127.8, 104.5)
- removed SW101 (x2): SW_DPDT_x2, Button_Switch_SMD:SW_DPDT_CK_JS202011JCQN
- removed the U3 at (117.1, 60.8)
- R1: value 30.1k -> 52.2k
- moved C8 106.8 mm to (117.2, 113.0), turned to 180 degrees
- moved C403 103.4 mm to (138.0, 106.0), turned to 180 degrees
- moved C9 102.5 mm to (132.0, 106.0), turned to 180 degrees
- moved C2 101.8 mm to (126.0, 73.0)
- moved C4 101.6 mm to (130.0, 70.0), turned to 90 degrees
- moved R4 101.5 mm to (134.0, 109.0), turned to 90 degrees
- moved C3 100.9 mm to (128.0, 70.0), turned to 90 degrees
- moved C107 100.8 mm to (131.0, 76.0), turned to 90 degrees
- moved C103 100.0 mm to (129.0, 76.0), turned to 90 degrees
- moved C102 99.3 mm to (127.0, 76.0), turned to 90 degrees
- moved C101 98.7 mm to (125.0, 76.0), turned to 90 degrees
- moved R3 95.6 mm to (125.0, 105.0), turned to 90 degrees
- moved C5 92.4 mm to (138.0, 83.0), turned to 180 degrees
- moved R5 92.3 mm to (127.0, 105.0), turned to -90 degrees
- moved C402 90.9 mm to (117.2, 101.0), turned to 180 degrees
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Connections:
- net DATA1 renamed /DATA1
- net DATA2 renamed /DATA2
- net NRST renamed /NRST
- net ST-RX renamed /ST_RX
- net ST_TX renamed /ST_TX
- net SWCLK renamed /SWCLK
- net SWDIO renamed /SWDIO
- net SWO renamed /SWO
- net VDD_SER renamed /VDD_SER
- C403 pad 1: /Regulation/Vin -> +BATT
- C404 pad 1: /Regulation/Vin -> +BATT
- C406 pad 1: /Regulation/12V -> +7.5V
- C5 pad 1: /Regulation/Vin -> +BATT
- R2 pad 1: /Regulation/12V -> +7.5V
- R407 pad 1: /Regulation/7.4V -> +7.5V
- U1 pad 10: SS -> /SS
- U1 pad 11: SCLK -> /SCLK
- U1 pad 12: MISO -> /MISO
- U1 pad 13: MOSI -> /MOSI
- U3 pad 1: MISO -> /MISO
- U3 pad 12: SCLK -> /SCLK
- U3 pad 14: MOSI -> /MOSI
