File: Capteurs_PCB/Capteurs_PCB.kicad_pcb (KiCad board)
At the start: 2 copper layers, 64 x 70 mm, 53 parts, among them J1 Conn_01x04, J101 Conn_01x03, J103 Conn_02x20_Odd_Even, J104 Conn_ST_STDC14, J2 Conn_01x03, J4 Conn_01x02, J6 Conn_01x03, J7 Conn_01x03, U1 STM32L412KBTx, U3 LSM6DSL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

Commit message: PCB
Routing:
- net GND: track 8.48 -> 14.9 mm, vias 1 -> 4
- net /MISO: track 20.7 -> 17.3 mm, vias 2 -> 0
- net /INT2: track 38.5 -> 41.5 mm
- net /Sig_LED: track 43.7 -> 46.1 mm, vias 0 -> 2
- net +BATT: track 105.5 -> 107.8 mm, vias 0 -> 2
- net /INT1: track 17.4 -> 19.6 mm, vias 0 -> 2
- net /ST_RX: track 29.5 -> 31.7 mm, vias 0 -> 2
- net +3.3V: track 161.1 -> 160.6 mm, vias 5 -> 7

Commit message: Finition et plus d'erreur sur le PCB
Parts:
- moved J101 40.4 mm to (145.6, 115.0), turned to 180 degrees
- moved C103 18.1 mm to (113.6, 68.7), turned to 180 degrees
- moved J2 7.63 mm to (107.1, 97.9)
- moved C107 6.48 mm to (125.5, 78.3), turned to -90 degrees
- moved C101 2.73 mm to (128.3, 77.9), turned to 0 degrees
- moved C102 0.75 mm to (128.3, 76.2), turned to 0 degrees
Routing:
- net /SigProp1: track 35.8 -> 74.2 mm
- net /NRST: track 48.6 -> 65.5 mm, vias 2 -> 4
- net +5V: track 119.1 -> 109.6 mm, vias 0 -> 2
- net /SigProp2: track 29.0 -> 37.1 mm
- net +3.3V: track 160.6 -> 167.1 mm
- net GND: track 14.9 -> 19.0 mm
