File: Capteurs_PCB/MPL115A1.kicad_sch (KiCad schematic)
At the start: 2 parts, among them U6 32350268

Commit message: Empreintes modifiées
Parts:
- C1: footprint Capacitor_SMD:C_1206_3216Metric -> Capacitor_SMD:C_1206_3216Metric_Pad1.33x1.80mm_HandSolder
Changed lines of the file:
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@@
       (effects (font (size 1.27 1.27)))
     )
-    (property "Footprint" "Capacitor_SMD:C_1206_3216Metric" (at 130.81 77.47 0)
+    (property "Footprint" "Capacitor_SMD:C_1206_3216Metric_Pad1.33x1.80mm_HandSolder" (at 130.81 77.47 0)
       (effects (font (size 1.27 1.27)) hide)
     )

Commit message: Footprint design and Footprint assignment
Parts:
- U6: footprint (none) -> Custom:Pressure_Captor_Custom
Changed lines of the file:
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@@
       (effects (font (size 1.27 1.27)) (justify left))
     )
-    (property "Footprint" "" (at 134.62 66.04 0)
+    (property "Footprint" "Custom:Pressure_Captor_Custom" (at 134.62 66.04 0)
       (effects (font (size 1.27 1.27)) hide)
     )

Commit message: Routage en cours
Parts:
- C1: footprint Capacitor_SMD:C_1206_3216Metric_Pad1.33x1.80mm_HandSolder -> Capacitor_SMD:C_0603_1608Metric_Pad1.08x0.95mm_HandSolder
Changed lines of the file:
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@@
       (effects (font (size 1.27 1.27)))
     )
-    (property "Footprint" "Capacitor_SMD:C_1206_3216Metric_Pad1.33x1.80mm_HandSolder" (at 130.81 77.47 0)
+    (property "Footprint" "Capacitor_SMD:C_0603_1608Metric_Pad1.08x0.95mm_HandSolder" (at 130.81 77.47 0)
       (effects (font (size 1.27 1.27)) hide)
     )
