File: Capteurs_PCB/regulation.kicad_sch (KiCad schematic)
At the start: 27 parts

Commit message: Suite PCB
Connections:
- net 7.4V is gone; now on net 7.5V: R407.1
Changed lines of the file:
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@@
     (effects (font (size 1.27 1.27)) (justify left bottom))
   )
-  (hierarchical_label "7.4V" (shape input) (at 185.42 64.77 90) (fields_autoplaced)
+  (hierarchical_label "7.5V" (shape input) (at 185.42 64.77 90) (fields_autoplaced)
     (effects (font (size 1.27 1.27)) (justify left))
   )
